Commit message: Clean up bringup package, update controller and description, add new models

File: control/bumperbot_ws/src/bumperbot_description/urdf/bumperbot.urdf.xacro (robot description, xacro)
@@ -1,6 +1,5 @@
 <?xml version="1.0"?>
 <robot name="bumperbot" xmlns:xacro="http://ros.org/wiki/xacro">
-  <!-- Load Simulated or Real Hardware Interfaces -->
-  <xacro:arg name="is_sim" default="true"/>
+  <xacro:arg name="is_ignition" default="true"/>
   <!-- Include Gazebo Parameters -->
   <xacro:include filename="$(find bumperbot_description)/urdf/bumperbot_gazebo.xacro" />
@@ -143,5 +142,5 @@
     <axis xyz="0 0 0" />
   </joint>
-  <link name="can_link">
+  <!--  <link name="can_link">
     <visual>
         <origin rpy="1.57 0 0" xyz="-0.03 0.03 0"/>
@@ -155,5 +154,5 @@
       <child link="can_link"/>
       <origin rpy="0 0 0" xyz="0 0 0.078"/>
-  </joint>
+  </joint> -->
   <link name="imu_link">
     <inetrial>

File: control/bumperbot_ws/src/bumperbot_description/urdf/bumperbot_gazebo.xacro (robot description, xacro)
@@ -54,9 +54,16 @@
   <!-- ROS 2 Control -->
   <gazebo>
-    <plugin filename="libgazebo_ros2_control.so" name="gazebo_ros2_control">
-      <robot_param>robot_description</robot_param>
-      <robot_param_node>robot_state_publisher</robot_param_node>
-      <parameters>$(find bumperbot_controller)/config/bumperbot_controllers.yaml</parameters>
-    </plugin>
+    <!-- ROS 2 Humble -->
+    <xacro:if value="$(arg is_ignition)">
+      <plugin filename="ign_ros2_control-system" name="ign_ros2_control::IgnitionROS2ControlPlugin">
+        <parameters>$(find bumperbot_controller)/config/bumperbot_controllers.yaml</parameters>
+      </plugin>
+    </xacro:if>
+    <!-- ROS 2 Iron or above -->
+    <xacro:unless value="$(arg is_ignition)">
+      <plugin filename="gz_ros2_control-system" name="gz_ros2_control::GazeboSimROS2ControlPlugin">
+        <parameters>$(find bumperbot_controller)/config/bumperbot_controllers.yaml</parameters>
+      </plugin>
+    </xacro:unless>
   </gazebo>
   <!--IMU-->

File: control/bumperbot_ws/src/bumperbot_description/urdf/bumperbot_ros2_control.xacro (robot description, xacro)
@@ -2,14 +2,13 @@
 <robot xmlns:xacro="http://www.ros.org/wiki/xacro" name="bumperbot">
     <ros2_control name="RobotSystem" type="system">
-        <xacro:if value="$(arg is_sim)">
-            <!-- ros2_control Gazebo -->
+        <!-- ros2_control Gazebo -->
+        <xacro:if value="$(arg is_ignition)">
             <hardware>
-                <plugin>gazebo_ros2_control/GazeboSystem</plugin>
+                <plugin>ign_ros2_control/IgnitionSystem</plugin>
             </hardware>
         </xacro:if>
-        <xacro:unless value="$(arg is_sim)">
+        <xacro:unless value="$(arg is_ignition)">
             <hardware>
-                <plugin>bumperbot_firmware/BumperbotInterface</plugin>
-                <param name="port">/dev/ttyUSB0</param>
+                <plugin>gz_ros2_control/GazeboSimSystem</plugin>
             </hardware>
         </xacro:unless>
