Commit message: laser-link

File: SLAM/bumperbot_ws/src/bumperbot_description/urdf/bumperbot.urdf.xacro (robot description, xacro)
@@ -155,4 +155,28 @@
       <origin rpy="0 0 0" xyz="0 0 0.078"/>
   </joint> -->
+  <link name="laser_link">
+    <inertial>
+      <origin xyz="-0.011945780406062 -0.000381929217680526 -0.0170649378129477" rpy="0 0 0" />
+      <mass value="0.073084435549317" />
+      <inertia ixx="1.96074931730795E-05" ixy="-3.62091076640009E-07" ixz="4.28230084046735E-07" iyy="2.40983835136327E-05" iyz="1.50180909250652E-08" izz="4.14184164228595E-05" />
+    </inertial>
+    <visual>
+      <origin xyz="0 0 0" rpy="0 0 0"/>
+      <geometry>
+        <mesh filename="package://bumperbot_description/meshes/laser_link.STL"/>
+      </geometry>
+    </visual>
+    <collision>
+      <origin xyz="0 0 0" rpy="0 0 0"/>
+        <geometry>
+          <mesh filename="package://bumperbot_description/meshes/laser_link.STL"/>
+        </geometry>
+    </collision>
+  </link>
+  <joint name="laser_joint" type="fixed">
+    <parent link="base_link"/>
+    <child link="laser_link"/>
+    <origin xyz="0.0 0.0 0.1208" rpy="0 0 3.14" />
+  </joint>
   <link name="imu_link">
     <inetrial>

File: SLAM/bumperbot_ws/src/bumperbot_description/urdf/bumperbot_gazebo.xacro (robot description, xacro)
@@ -59,4 +59,9 @@
         <parameters>$(find bumperbot_controller)/config/bumperbot_controllers.yaml</parameters>
       </plugin>
+      <plugin filename="ignition-gazebo-imu-system" name="ignition::gazebo::systems::Imu">
+      </plugin>
+      <plugin filename="ignition-gazebo-sensors-system" name="ignition::gazebo::systems::Sensors">
+        <render_engine>orge2</render_engine>
+      </plugin>
     </xacro:if>
     <!-- ROS 2 Iron or above -->
@@ -64,4 +69,9 @@
       <plugin filename="gz_ros2_control-system" name="gz_ros2_control::GazeboSimROS2ControlPlugin">
         <parameters>$(find bumperbot_controller)/config/bumperbot_controllers.yaml</parameters>
+      </plugin>
+      <plugin filename="gz-sim-imu-system" name="gz::sim::systems::Imu">
+      </plugin>
+      <plugin filename="gz-sim-sensors-system" name="gz::sim::systems::Sensors">
+        <render_engine>orge2</render_engine>
       </plugin>
     </xacro:unless>
@@ -119,3 +129,32 @@
     </sensor>
   </gazebo>
+  <gazebo reference="laser_link">
+    <sensor name="lidar" type="gpu_ray">
+      <always_on>true</always_on>
+      <vizualize>true</vizualize>
+      <topic>scan</topic>
+      <update_rate>5</update_rate>
+      <gz_frame_id>laser_link</gz_frame_id>
+      <ray>
+        <scan>
+          <horizontal>
+            <samples>360</samples>
+            <resolution>1.0</resolution>
+            <min_angle>0.0</min_angle>
+            <max_angle>6.28</max_angle>
+          </horizontal>
+        </scan>
+        <range>
+          <min>0.12</min>
+          <max>12.0</max>
+          <resolution>0.02</resolution>
+        </range>
+        <noise>
+          <type>gaussian</type>
+          <mean>0.0</mean>
+          <stddev>0.01</stddev>
+        </noise>
+      </ray>
+    </sensor>
+  </gazebo>
 </robot>
